File: KiCad/control_board/control_board.kicad_pcb (KiCad board)
At the start: 2 copper layers, 375 x 40 mm, 80 parts, among them J1 Conn_01x02_Male, J2 USB_B, J3 Conn_01x04_Male, J4 Conn_01x03_Male, J5 DS1013-06S, J6 Conn_01x06_Male, Q1 BSS84, SW1 SW_Push, SW10 SW_Push, SW11 SW_Push, SW12 Rotary_Encoder, SW2 SW_Push, SW3 SW_Push, SW4 SW_Push, SW5 SW_Push, SW6 SW_Push, SW7 SW_Push, SW8 SW_Push, SW9 SW_Push, U1 ATmega32U4-AU, U2 74HC595, U3 USBLC6-2SC6, Y1 Crystal_GND24

Commit message: Adding 2 more channels.
Parts:
- removed F1: MF-MSMF050-2, Fuse:Fuse_1812_4532Metric_Pad1.30x3.40mm_HandSolder
- removed Q1: BSS84, Package_TO_SOT_SMD:SOT-23
- removed the R23 at (96.6, 133.1)
- removed the REF** at (366.0, 114.0)
- removed the REF** at (110.0, 114.0)
- removed the REF** at (366.0, 134.0)
- removed the REF** at (213.0, 114.0)
- removed the SW12 at (60.4, 148.3)
- added C10: 0.1u, Capacitor_SMD:C_0805_2012Metric, F.Cu at (336.2, 125.2)
- added C11: 0.1u, Capacitor_SMD:C_0805_2012Metric, F.Cu at (45.7, 120.2)
- added C7: 0.1u, Capacitor_SMD:C_0805_2012Metric, F.Cu at (232.9, 113.8)
- added C8: 0.1u, Capacitor_SMD:C_0805_2012Metric, F.Cu at (245.7, 113.8)
- added C9: 0.1u, Capacitor_SMD:C_0805_2012Metric, F.Cu at (350.2, 125.2)
- added D10: LED, LED_THT:LED_D3.0mm_Horizontal_O6.35mm_Z10.0mm, F.Cu at (382.7, 137.5)
- added D9: LED, LED_THT:LED_D3.0mm_Horizontal_O6.35mm_Z10.0mm, F.Cu at (368.7, 137.5)
- added J7: EXT, Connector_JST:JST_PH_B7B-PH-K_1x07_P2.00mm_Vertical, F.Cu at (112.7, 112.5)
- added R10: 1k, Resistor_SMD:R_0805_2012Metric, F.Cu at (381.3, 132.2)
- added R16: 2k, Resistor_SMD:R_0805_2012Metric, F.Cu at (263.2, 116.7)
- added R24: 39k, Resistor_SMD:R_0805_2012Metric, F.Cu at (96.2, 136.0)
- added R39: 39k, Resistor_SMD:R_0805_2012Metric, F.Cu at (373.1, 132.2)
- added R40: 39k, Resistor_SMD:R_0805_2012Metric, F.Cu at (387.0, 132.2)
- added R9: 1k, Resistor_SMD:R_0805_2012Metric, F.Cu at (367.3, 132.2)
- added REF**: MountingHole_3.5mm, MountingHole:MountingHole_3.5mm, F.Cu at (363.0, 114.0)
- added REF**: MountingHole_3.5mm, MountingHole:MountingHole_3.5mm, F.Cu at (363.0, 137.0)
- added SW10: SW_Push, Button_Switch_THT:SW_Tactile_SPST_Angled_PTS645Vx83-2LFS, F.Cu at (386.2, 144.4)
- added SW11: SW_Push, Button_Switch_THT:SW_Tactile_SPST_Angled_PTS645Vx83-2LFS, F.Cu at (231.2, 144.4)
- added SW14: Rotary_Encoder, PEC16:RotaryEncoder_Bourns_PEC16-2215F-N0024_Vertical, F.Cu at (64.0, 149.4)
- added U4: 74HC165, Package_SO:SOIC-16_3.9x9.9mm_P1.27mm, F.Cu at (236.5, 120.2)
- added U5: 74HC165, Package_SO:SOIC-16_3.9x9.9mm_P1.27mm, F.Cu at (249.2, 120.2)
- added U6: 74HC595, Package_SO:SOIC-16_3.9x9.9mm_P1.27mm, F.Cu at (343.2, 120.2)
- added U7: 74HC595, Package_SO:SOIC-16_3.9x9.9mm_P1.27mm, F.Cu at (329.2, 120.2)
- added U8: AT25640B, Package_SO:SO-8_3.9x4.9mm_P1.27mm, F.Cu at (43.1, 125.8)
- J1: value Conn_01x02_Male -> +5V GND
- J2: value USB_B -> REL; footprint Connector_USB:USB_B_OST_USB-B1HSxx_Horizontal -> Connector_JST:JST_PH_B11B-PH-K_1x11_P2.00mm_Vertical
- J3: value Conn_01x04_Male -> GND VBUS USB; footprint Connector_JST:JST_EH_B4B-EH-A_1x04_P2.50mm_Vertical -> Connector_JST:JST_PH_B4B-PH-K_1x04_P2.00mm_Vertical
- J4: value Conn_01x03_Male -> RX TX MUTE MIDI GND; footprint Connector_JST:JST_EH_B3B-EH-A_1x03_P2.50mm_Vertical -> Connector_JST:JST_PH_B5B-PH-K_1x05_P2.00mm_Vertical
- J6: value Conn_01x06_Male -> OLED; footprint Connector_JST:JST_EH_B6B-EH-A_1x06_P2.50mm_Vertical -> Connector_JST:JST_PH_B6B-PH-K_1x06_P2.00mm_Vertical
- Y1: value Crystal_GND24 -> Crystal_Small; footprint Crystal:Crystal_SMD_0603-4Pin_6.0x3.5mm_HandSoldering -> Crystal:Crystal_SMD_HC49-SD
- moved R12 304.9 mm to (74.6, 118.9), turned to 90 degrees
- moved U3 299.0 mm to (75.9, 113.2), turned to 270 degrees
- moved R13 296.0 mm to (77.2, 118.9), turned to 90 degrees
- moved J4 222.9 mm to (96.8, 112.5)
- moved SW9 141.3 mm to (372.2, 144.4)
- moved J2 60.4 mm to (325.0, 112.5), turned to 0 degrees
- moved J1 47.6 mm to (47.9, 112.5)
- moved J6 32.2 mm to (129.9, 127.8), turned to 180 degrees
- moved R21 26.9 mm to (77.2, 144.3), turned to 270 degrees
- moved R15 25.5 mm to (41.0, 116.3), turned to 270 degrees
- moved C3 22.3 mm to (91.8, 127.8), turned to 180 degrees
- moved C5 19.9 mm to (63.2, 127.1), turned to 270 degrees
- moved C4 15.6 mm to (71.4, 118.9), turned to 270 degrees
- moved C1 13.1 mm to (51.6, 135.4), turned to 180 degrees
- moved R14 12.2 mm to (91.8, 136.0), turned to 180 degrees
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- renumbered D9 to D11, R9 to R11, R10 to R12, R11 to R13, R13 to R15, R12 to R22, R24 to R23, SW10 to SW12, SW11 to SW13
Connections:
- J1 pad 1: RX -> +5V
- J1 pad 2: TX -> GND
- J2 pad 1: Net-(F1-Pad2) -> LOOP8
- J2 pad 2: Net-(J2-Pad2) -> LOOP9
- J2 pad 3: Net-(J2-Pad3) -> LOOP10
- J2 pad 4: GND -> LOOP1
- J2 pad 5: GND -> LOOP2
- J3 pad 1: +9V -> GND
- J3 pad 2: GND -> VBUS
- J3 pad 3: GND -> Net-(J3-Pad3)
- J3 pad 4: +5V -> Net-(J3-Pad4)
- J4 pad 1: SCK -> RX
- J4 pad 2: REL_SER -> TX
- J4 pad 3: REL_CS -> MUTE
- R12 pad 2: Net-(R10-Pad2) -> Net-(R12-Pad2)
- R13 pad 2: Net-(R11-Pad2) -> Net-(R13-Pad2)
- SW9 pad 1: SW_STORE -> SW9
- U1 pad 1: SW5 -> Net-(U1-Pad1)
- U1 pad 18: Net-(U1-Pad18) -> EXT_IO
- U1 pad 19: SW1 -> EXT_CS
- U1 pad 22: SW3 -> EEPROM_CS
- U1 pad 25: SW2 -> SW_LEFT
- U1 pad 26: SW3 -> SW_RIGHT
- U1 pad 27: SW4 -> Net-(U1-Pad27)
- U1 pad 31: Net-(U1-Pad31) -> SW_CS
- U1 pad 32: STORE_LED -> D_STORE
- U1 pad 36: SW_RIGHT -> Net-(U1-Pad36)
- U1 pad 37: SW_LEFT -> Net-(U1-Pad37)
- U1 pad 39: SW8 -> Net-(U1-Pad39)
- U1 pad 40: SW7 -> MIDI_MODE
- U1 pad 41: SW6 -> MUTE
- U1 pad 8: MUTE -> Net-(U1-Pad8)
- U2 pad 1: D2 -> D1
- U2 pad 11: REL_CS -> SCK
- U2 pad 12: SCK -> REL_CS
- U2 pad 13: +5V -> GND
- U2 pad 15: D1 -> Net-(U2-Pad15)
- U2 pad 2: D3 -> D2
- U2 pad 3: D4 -> D3
- U2 pad 4: D5 -> D4
- U2 pad 5: D6 -> D5
- U2 pad 6: D7 -> D6
- U2 pad 7: D8 -> D7
- U2 pad 9: REL_SER -> SER2
- U3 pad 1: Net-(J2-Pad3) -> Net-(J3-Pad3)
- U3 pad 3: Net-(J2-Pad2) -> Net-(J3-Pad4)
- U3 pad 4: Net-(R11-Pad2) -> Net-(R12-Pad2)
- U3 pad 6: Net-(R10-Pad2) -> Net-(R13-Pad2)
- Y1 pad 2: GND -> Net-(C2-Pad1)
Routing:
- net +5V: track 0.00 -> 721.1 mm, vias 0 -> 23
- net SCK: track 0.00 -> 343.6 mm, vias 0 -> 10
- net MOSI: track 0.00 -> 299.4 mm, vias 0 -> 7
- net REL_CS: track 0.00 -> 293.6 mm, vias 0 -> 4
- net GND: track 0.00 -> 209.7 mm, vias 0 -> 12
- net SW10: track 0.00 -> 180.9 mm
- net SW_CS: track 0.00 -> 180.9 mm, vias 0 -> 3
- net SW_STORE: track 0.00 -> 173.6 mm, vias 0 -> 1
- net D_STORE: track 0.00 -> 166.5 mm, vias 0 -> 1
- net SW9: track 0.00 -> 165.7 mm
- net SW8: track 0.00 -> 150.5 mm
- net SW7: track 0.00 -> 135.2 mm
- net MISO: track 0.00 -> 121.1 mm, vias 0 -> 5
- net SW6: track 0.00 -> 117.5 mm
- net SW5: track 0.00 -> 100.6 mm
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- added copper zone on B.Cu, net GND
- added copper zone on F.Cu, net GND
Other:
- outline, holes or cut-outs redrawn
- net class Medium added: clearance 0.2, trace_width 0.3, via_dia 0.8, via_drill 0.4
- net class Thick added: clearance 0.2, trace_width 0.4, via_dia 0.8, via_drill 0.4

Commit message: RC1
Parts:
- removed R16: 2k, Resistor_SMD:R_0805_2012Metric
- added C12: 0.1u, Capacitor_SMD:C_0805_2012Metric, F.Cu at (258.6, 123.1)
- added D12: LED, LED_THT:LED_D3.0mm_Horizontal_O6.35mm_Z10.0mm, F.Cu at (22.7, 140.5)
- added D13: LED, LED_THT:LED_D3.0mm_Horizontal_O6.35mm_Z10.0mm, F.Cu at (108.7, 140.5)
- added R17: 1k, Resistor_SMD:R_0805_2012Metric, F.Cu at (32.0, 136.0)
- added R18: 1k, Resistor_SMD:R_0805_2012Metric, F.Cu at (104.0, 136.0)
- added U9: SN74LVC1G125DBVR, Package_TO_SOT_SMD:SOT-23-5, F.Cu at (258.8, 118.8)
- J1: value +5V GND -> JST B2B-XH-A; footprint Connector_JST:JST_EH_B2B-EH-A_1x02_P2.50mm_Vertical -> Connector_JST:JST_XH_B2B-XH-A_1x02_P2.50mm_Vertical
- J4: value RX TX MUTE MIDI GND -> JST B5B-PH-K-S
- moved J1 0.64 mm to (47.9, 113.2)
Connections:
- U1 pad 27: Net-(U1-Pad27) -> D_MIDI
Routing:
- net MISO: track 121.1 -> 264.0 mm, vias 5 -> 7
- net D_MIDI: track 0.00 -> 90.1 mm, vias 0 -> 1
- net EXT_IO: track 0.00 -> 70.2 mm, vias 0 -> 2
- net EXT_CS: track 0.00 -> 68.8 mm, vias 0 -> 2
- net +5V: track 721.1 -> 745.6 mm, vias 23 -> 24
- net SW_CS: track 180.9 -> 203.0 mm, vias 3 -> 4
- net Net-(D12-Pad1): track 0.00 -> 10.9 mm
- net SCK: track 343.6 -> 350.6 mm, vias 10 -> 11
- net Net-(D13-Pad1): track 0.00 -> 6.79 mm
- net Net-(U5-Pad9): track 0.00 -> 6.63 mm
- net MOSI: track 299.4 -> 304.8 mm
- net OLED_CS: track 58.7 -> 57.2 mm
- net GND: track 209.7 -> 210.9 mm, vias 12 -> 11
- net D_STORE: track 166.5 -> 166.0 mm

Commit message: Ready for production 2020.04.16
Parts:
- added G***: LOGO, bg:mpm_b, B.Cu at (207.6, 129.9)
- added G***: LOGO, bg:mpm_f, F.Cu at (178.8, 118.5)
- added J8: Conn_01x02_Male, Connector_PinHeader_2.54mm:PinHeader_1x02_P2.54mm_Vertical, F.Cu at (42.5, 112.5)
- added REF**: MountingHole_3.5mm, MountingHole:MountingHole_3.5mm, F.Cu at (307.0, 137.0)
- added REF**: MountingHole_3.5mm, MountingHole:MountingHole_3.5mm, F.Cu at (243.0, 134.0)
- added REF**: KiCad-Logo2_8mm_SilkScreen, Symbol:KiCad-Logo2_8mm_SilkScreen, F.Cu at (377.8, 120.3)
- J2: value REL -> JST B11B-PH-K-S
- J3: value GND VBUS USB -> JST B4B-PH-K-S
- J6: value OLED -> JST B6B-PH-K-S
- J7: value EXT -> JST B7B-PH-K-S
- SW14: value Rotary_Encoder -> PEC16-2215F-N0024
- Y1: value Crystal_Small -> HC-49SM
- moved R15 24.3 mm to (64.7, 121.7), turned to 0 degrees
- moved Y1 1.40 mm to (58.9, 132.7)
- moved REF** 1.00 mm to (285.0, 114.0)
- moved C5 0.74 mm to (63.8, 126.8)
Connections:
- J5 pad 2: +5V -> ISCP_5V
Routing:
- net +5V: track 745.6 -> 735.2 mm
- net ISCP_5V: track 0.00 -> 7.28 mm
- net TX: track 50.6 -> 57.6 mm
- net MOSI: track 304.8 -> 300.3 mm, vias 7 -> 6
- net RX: track 47.7 -> 51.9 mm
- net EEPROM_CS: track 38.8 -> 41.7 mm
- net GND: track 210.9 -> 213.6 mm, vias 11 -> 12
- net RST: track 46.7 -> 44.2 mm, vias 2 -> 1
- net SW8: track 150.5 -> 152.8 mm
- net SW10: track 180.9 -> 183.3 mm
- net SW9: track 165.7 -> 168.0 mm
- net SW7: track 135.2 -> 137.6 mm
- net SW_CS: track 203.0 -> 201.8 mm
- net D_STORE: track 166.0 -> 165.0 mm
- net MISO: track 264.0 -> 263.1 mm, vias 7 -> 6
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Other:
- board text added: "2020.04.16"
- board text added: "github.com/mar0x/patch_mate"
