File: KiCad/relay_board/relay_board.kicad_pcb (KiCad board)
At the start: 2 copper layers, 385 x 50 mm, 82 parts, among them J1 DIN-5-OOTDTY, J2 DIN-5-OOTDTY, J3 DIN-5-OOTDTY, J4 DS-210, J5 Conn_01x06_Male, J6 Conn_01x05_Male, J7 Conn_01x04_Male, J8 Conn_01x03_Male, J9 USB_B, Q1 BC817, Q2 BSS84, Q3 BSS84, U1 ULN2803A, U2 LM2575-5.0BU, U3 LM2575-5.0BT, U4 6N138, U5 74AUC1G125, U6 74HC595

Commit message: Adding 2 more channels.
Parts:
- removed D1, D2: D, Diode_SMD:D_SMA
- removed Q1: BC817, Package_TO_SOT_SMD:SOT-23
- removed R5: 220, Resistor_SMD:R_0805_2012Metric
- added F1: MF-MSMF050-2, Fuse:Fuse_1812_4532Metric_Pad1.30x3.40mm_HandSolder, F.Cu at (75.6, 91.0)
- added J10: REL, Connector_JST:JST_PH_B11B-PH-K_1x11_P2.00mm_Vertical, F.Cu at (374.7, 116.4)
- added K_MIDI_OUT1: G6K-2, Relay_SMD:Relay_DPDT_Omron_G6K-2F-Y, F.Cu at (113.7, 103.7)
- added K_RET10: G6K-2, Relay_SMD:Relay_DPDT_Omron_G6K-2F-Y, F.Cu at (181.3, 101.1)
- added K_RET9: G6K-2, Relay_SMD:Relay_DPDT_Omron_G6K-2F-Y, F.Cu at (202.9, 101.1)
- added K_SEND10: G6K-2, Relay_SMD:Relay_DPDT_Omron_G6K-2F-Y, F.Cu at (192.1, 101.1)
- added K_SEND9: G6K-2, Relay_SMD:Relay_DPDT_Omron_G6K-2F-Y, F.Cu at (213.7, 101.1)
- added LOOP10: AudioJack3_Dual_Switch, CK635-037:CK635-037, F.Cu at (190.0, 70.0)
- added LOOP9: AudioJack3_Dual_Switch, CK635-037:CK635-037, F.Cu at (210.0, 70.0)
- added U7: 74AUC1G125, Package_TO_SOT_SMD:SOT-23-5, F.Cu at (104.2, 97.3)
- D3: value D_Bridge_+-AA -> D_Bridge_+AA-; footprint Diode_SMD:Diode_Bridge_Vishay_DFS -> DiodeBridge:Diode_Bridge_KBP20x
- J1: value DIN-5-OOTDTY -> MIDI IN
- J2: value DIN-5-OOTDTY -> MIDI THRU
- J3: value DIN-5-OOTDTY -> MIDI OUT
- J5: value Conn_01x06_Male -> +5V GND; footprint Connector_JST:JST_EH_B6B-EH-A_1x06_P2.50mm_Vertical -> Connector_JST:JST_EH_B2B-EH-A_1x02_P2.50mm_Vertical
- J6: value Conn_01x05_Male -> RX TX MUTE MIDI GND; footprint Connector_JST:JST_EH_B5B-EH-A_1x05_P2.50mm_Vertical -> Connector_JST:JST_PH_B5B-PH-K_1x05_P2.00mm_Vertical
- J7: value Conn_01x04_Male -> USB; footprint Connector_JST:JST_EH_B4B-EH-A_1x04_P2.50mm_Vertical -> Connector_JST:JST_PH_B4B-PH-K_1x04_P2.00mm_Vertical
- J8: value Conn_01x03_Male -> BTN LED; footprint Connector_JST:JST_EH_B3B-EH-A_1x03_P2.50mm_Vertical -> Connector_JST:JST_EH_B4B-EH-A_1x04_P2.50mm_Vertical
- U1: value ULN2803A -> ULN2003; footprint Package_SO:SOIC-18W_7.5x11.6mm_P1.27mm -> Package_SO:SOIC-16_3.9x9.9mm_P1.27mm
- U6: value 74HC595 -> ULN2003
- moved J6 170.9 mm to (146.8, 116.4)
- moved U6 139.7 mm to (244.2, 113.8)
- moved C3 131.8 mm to (252.7, 111.4), turned to 180 degrees
- moved J5 123.1 mm to (98.0, 117.0)
- moved LOOP5 86.1 mm to (320.0, 70.0)
- moved K_RET5 80.5 mm to (311.5, 101.1)
- moved K_SEND5 80.0 mm to (322.3, 101.1)
- moved K_RET8 67.1 mm to (224.5, 101.1)
- moved K_SEND8 66.7 mm to (235.3, 101.1)
- moved K_RET7 66.3 mm to (246.1, 101.1)
- moved K_RET4 65.8 mm to (333.1, 101.1)
- moved K_SEND7 65.8 mm to (256.9, 101.1)
- moved J1 65.6 mm to (132.5, 82.7)
- moved K_SEND4 65.4 mm to (343.8, 101.1)
- moved K_RET6 65.4 mm to (267.6, 101.1)
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Connections:
- D3 pad 2: GND -> Net-(D3-Pad2)
- D3 pad 4: Net-(D3-Pad4) -> GND
- INOUT5 pad R1: LOOP4_R -> LOOP5_R
- INOUT5 pad R2: LOOP5_R -> LOOP6_R
- INOUT5 pad RN2: LOOP4_R -> LOOP5_R
- INOUT5 pad S1: GNDA -> GND
- INOUT5 pad S2: GNDA -> GND
- INOUT5 pad SN1: GNDA -> GND
- INOUT5 pad SN2: GNDA -> GND
- INOUT5 pad T1: LOOP4_T -> LOOP5_T
- INOUT5 pad T2: LOOP5_T -> LOOP6_T
- INOUT5 pad TN2: LOOP4_T -> LOOP5_T
- J4 pad 1: Net-(D3-Pad3) -> Net-(D3-Pad2)
- J4 pad 2: Net-(D3-Pad4) -> Net-(D3-Pad3)
- J5 pad 1: +9V -> +5V
- J6 pad 1: +5V -> RX
- J6 pad 2: SCK -> TX
- J6 pad 3: REL_SER -> MUTE
- J6 pad 4: REL_CS -> MIDI_MODE
- J8 pad 1: GND -> +5V
- J9 pad 1: VBUS -> Net-(F1-Pad1)
- K_MUTE1 pad 2: LOOP4_T -> LOOP5_T
- K_MUTE1 pad 7: LOOP4_R -> LOOP5_R
- K_MUTE2 pad 2: LOOP8_T -> LOOP10_T
- K_MUTE2 pad 7: LOOP8_R -> LOOP10_R
- K_RET4 pad 3: LOOP4_T -> Net-(K_RET4-Pad3)
- K_RET4 pad 6: LOOP4_R -> Net-(K_RET4-Pad6)
- K_RET5 pad 3: Net-(K_RET5-Pad3) -> LOOP5_T
- K_RET5 pad 6: Net-(K_RET5-Pad6) -> LOOP5_R
- K_RET8 pad 3: LOOP8_T -> Net-(K_RET8-Pad3)
- K_RET8 pad 6: LOOP8_R -> Net-(K_RET8-Pad6)
- K_SEND5 pad 3: LOOP5_T -> Net-(K_RET4-Pad3)
- K_SEND5 pad 6: LOOP5_R -> Net-(K_RET4-Pad6)
- K_SEND6 pad 3: Net-(K_RET5-Pad3) -> LOOP6_T
- K_SEND6 pad 6: Net-(K_RET5-Pad6) -> LOOP6_R
- LOOP1 pad S1: GNDA -> GND
- LOOP1 pad S2: GNDA -> GND
- LOOP1 pad SN1: GNDA -> GND
- LOOP1 pad SN2: GNDA -> GND
- LOOP2 pad S1: GNDA -> GND
- LOOP2 pad S2: GNDA -> GND
- LOOP2 pad SN1: GNDA -> GND
- LOOP2 pad SN2: GNDA -> GND
- LOOP3 pad S1: GNDA -> GND
- LOOP3 pad S2: GNDA -> GND
- LOOP3 pad SN1: GNDA -> GND
- LOOP3 pad SN2: GNDA -> GND
- LOOP4 pad S1: GNDA -> GND
- LOOP4 pad S2: GNDA -> GND
- LOOP4 pad SN1: GNDA -> GND
- LOOP4 pad SN2: GNDA -> GND
- LOOP5 pad S1: GNDA -> GND
- LOOP5 pad S2: GNDA -> GND
- LOOP5 pad SN1: GNDA -> GND
- LOOP5 pad SN2: GNDA -> GND
- LOOP6 pad S1: GNDA -> GND
- LOOP6 pad S2: GNDA -> GND
- LOOP6 pad SN1: GNDA -> GND
- LOOP6 pad SN2: GNDA -> GND
- LOOP7 pad S1: GNDA -> GND
- LOOP7 pad S2: GNDA -> GND
- LOOP7 pad SN1: GNDA -> GND
- LOOP7 pad SN2: GNDA -> GND
- LOOP8 pad S1: Net-(LOOP8-PadS1) -> GND
- LOOP8 pad S2: Net-(LOOP8-PadS1) -> GND
- LOOP8 pad SN1: Net-(LOOP8-PadS1) -> GND
- LOOP8 pad SN2: Net-(LOOP8-PadS1) -> GND
- MAIN_IN1 pad S: GNDA -> GND
- MAIN_IN1 pad SN: GNDA -> GND
- MAIN_IN2 pad S: GNDA -> GND
- MAIN_OUT1 pad R: LOOP8_R -> LOOP10_R
- MAIN_OUT1 pad S: GNDA -> GND
- MAIN_OUT1 pad SN: GNDA -> GND
- MAIN_OUT1 pad T: LOOP8_T -> LOOP10_T
- MAIN_OUT2 pad R: LOOP8_R -> LOOP10_R
- MAIN_OUT2 pad S: GNDA -> GND
- MAIN_OUT2 pad T: LOOP8_T -> LOOP10_T
- R1 pad 1: GNDA -> GND
- R12 pad 2: TX -> Net-(R12-Pad2)
- R2 pad 1: GNDA -> GND
- R3 pad 1: GNDA -> GND
- R4 pad 1: GNDA -> GND
- U1 pad 10: +5V -> REL7
- U1 pad 11: REL8 -> REL6
- U1 pad 12: REL7 -> REL5
- U1 pad 13: REL6 -> REL4
- U1 pad 14: REL5 -> REL3
- U1 pad 15: REL4 -> REL2
- U1 pad 16: REL3 -> REL1
- U1 pad 8: LOOP8 -> GND
- U1 pad 9: GND -> +5V
- U5 pad 5: VCC -> +5V
- U6 pad 1: LOOP1 -> MIDI_MODE
- U6 pad 10: +5V -> Net-(U6-Pad10)
- U6 pad 11: REL_CS -> Net-(U6-Pad11)
- U6 pad 12: SCK -> REL_MUTE
- U6 pad 13: +5V -> REL8
- U6 pad 14: REL_SER -> REL9
- U6 pad 15: LOOP8 -> REL10
- U6 pad 16: +5V -> REL_MIDI_MODE
- U6 pad 2: LOOP2 -> LOOP10
- U6 pad 3: LOOP3 -> LOOP9
- U6 pad 4: LOOP4 -> LOOP8
- U6 pad 5: LOOP5 -> MUTE
- U6 pad 6: LOOP6 -> Net-(U6-Pad6)
- U6 pad 7: LOOP7 -> Net-(U6-Pad7)
- U6 pad 9: Net-(U6-Pad9) -> +5V
Routing:
- net +5V: track 0.00 -> 1011.3 mm, vias 0 -> 29
- net REL7: track 0.00 -> 185.0 mm
- net REL6: track 0.00 -> 160.6 mm
- net REL_MUTE: track 0.00 -> 155.3 mm, vias 0 -> 2
- net LOOP10: track 0.00 -> 143.3 mm
- net LOOP9: track 0.00 -> 139.7 mm
- net LOOP8: track 0.00 -> 135.4 mm
- net REL_MIDI_MODE: track 0.00 -> 125.9 mm, vias 0 -> 2
- net REL5: track 0.00 -> 115.2 mm
- net MUTE: track 0.00 -> 96.2 mm
- net REL4: track 0.00 -> 91.9 mm
- net MIDI_MODE: track 0.00 -> 88.2 mm
- net PWR: track 0.00 -> 83.8 mm
- net RX: track 0.00 -> 78.9 mm
- net REL3: track 0.00 -> 68.7 mm
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- added copper zone on B.Cu, net GND
- added copper zone on F.Cu, net GND
Other:
- board size 385 x 50 mm -> 410 x 50 mm
- net class Medium added: clearance 0.2, trace_width 0.3, via_dia 0.8, via_drill 0.4
- net class Thick added: clearance 0.2, trace_width 0.4, via_dia 0.8, via_drill 0.4

Commit message: RC1
Parts:
- removed K_MIDI_OUT1: G6K-2, Relay_SMD:Relay_DPDT_Omron_G6K-2F-Y
- added C5: 0.1u, Capacitor_SMD:C_0805_2012Metric, F.Cu at (120.1, 97.3)
- added C6: 0.1u, Capacitor_SMD:C_0805_2012Metric, F.Cu at (111.2, 102.4)
- added C7: 0.1u, Capacitor_SMD:C_0805_2012Metric, F.Cu at (101.0, 97.3)
- added G***: LOGO, bg:mpm_f, F.Cu at (198.4, 113.6)
- added G***: LOGO, bg:mpm3, B.Cu at (240.1, 94.9)
- added R5: 39k, Resistor_SMD:R_0805_2012Metric, F.Cu at (113.7, 97.3)
- added REF**: KiCad-Logo2_8mm_SilkScreen, Symbol:KiCad-Logo2_8mm_SilkScreen, F.Cu at (350.3, 112.9)
- added U8: SN74LVC1G125DBVR, Package_TO_SOT_SMD:SOT-23-5, F.Cu at (105.5, 97.3)
- D3: value D_Bridge_+AA- -> RS202-BP
- D5: value 1N5819 -> 1N5822; footprint Diode_THT:D_DO-41_SOD81_P7.62mm_Horizontal -> Diode_THT:D_DO-201AD_P15.24mm_Horizontal
- J1: value MIDI IN -> DIN5MIDI-OOTDTY
- J10: value REL -> JST B11B-PH-K-S
- J2: value MIDI THRU -> DIN5MIDI-OOTDTY
- J3: value MIDI OUT -> DIN5MIDI-OOTDTY
- J5: value +5V GND -> JST B2B-XH-A; footprint Connector_JST:JST_EH_B2B-EH-A_1x02_P2.50mm_Vertical -> Connector_JST:JST_XH_B2B-XH-A_1x02_P2.50mm_Vertical
- J6: value RX TX MUTE MIDI GND -> JST B5B-PH-K-S
- J7: value USB -> JST B4B-PH-K-S
- J8: value BTN LED -> JST B4B-XH-A; footprint Connector_JST:JST_EH_B4B-EH-A_1x04_P2.50mm_Vertical -> Connector_JST:JST_XH_B4B-XH-A_1x04_P2.50mm_Vertical
- J9: value USB_B -> DS1099
- Q2, Q3: value BSS84 -> PMV65XP,215
- U5, U7: value 74AUC1G125 -> SN74LVC1G125DBVR
- moved R7 14.5 mm to (39.2, 91.3), turned to 270 degrees
- moved U7 12.5 mm to (115.6, 102.4)
- moved Q2 6.09 mm to (53.3, 87.4), turned to 180 degrees
- moved Q3 5.79 mm to (60.4, 87.4)
- moved D3 4.19 mm to (39.2, 84.6)
- moved C2 2.79 mm to (65.0, 101.1)
- moved C1 2.54 mm to (63.8, 112.0)
- moved D5 0.92 mm to (80.6, 109.9)
- moved J5 0.70 mm to (97.7, 116.4)
- moved J8 0.65 mm to (72.6, 116.4)
Connections:
- R12 pad 2: Net-(R12-Pad2) -> MIDI_OUT
- R7 pad 1: GND -> +9V
- R7 pad 2: +9V -> GND
- U5 pad 1: Net-(U5-Pad1) -> GND
- U6 pad 16: REL_MIDI_MODE -> ~MIDI_MODE
- U7 pad 1: Net-(U7-Pad1) -> MIDI_MODE
- U7 pad 2: MIDI_OUT -> TX
- U7 pad 4: Net-(R12-Pad2) -> MIDI_OUT
Routing:
- net ~MIDI_MODE: track 0.00 -> 140.8 mm, vias 0 -> 2
- net REL_MIDI_MODE: track 125.9 -> 0.00 mm, vias 2 -> 0
- net MIDI_MODE: track 88.2 -> 131.4 mm, vias 0 -> 1
- net LOOP10_T: track 38.4 -> 57.9 mm, vias 2 -> 0
- net +5V: track 1011.3 -> 1029.9 mm
- net LOOP5_T: track 48.2 -> 65.6 mm, vias 2 -> 0
- net RX: track 78.9 -> 92.5 mm
- net Net-(K_RET7-Pad2): track 17.6 -> 26.1 mm, vias 2 -> 0
- net VBUS: track 60.4 -> 68.8 mm
- net Net-(K_RET8-Pad2): track 17.7 -> 26.1 mm, vias 2 -> 0
- net Net-(K_RET9-Pad2): track 17.7 -> 26.1 mm, vias 2 -> 0
- net Net-(K_RET3-Pad2): track 17.8 -> 26.1 mm, vias 2 -> 0
- net Net-(K_RET2-Pad2): track 17.8 -> 26.1 mm, vias 2 -> 0
- net Net-(K_RET10-Pad2): track 17.8 -> 26.1 mm, vias 2 -> 0
- net Net-(K_RET4-Pad2): track 17.9 -> 26.1 mm, vias 2 -> 0
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Other:
- net class MegaThick added: clearance 0.2, trace_width 0.6, via_dia 0.8, via_drill 0.4
- board text added: "2020.03.26"

Commit message: Ready for production 2020.04.16
Parts:
- moved D3 2.81 mm to (42.0, 84.4)
Routing:
- net Net-(D3-Pad3): track 19.5 -> 16.6 mm
- net Net-(D3-Pad2): track 18.8 -> 16.1 mm
- net +9V: track 29.7 -> 28.6 mm
Other:
- board text added: "2020.04.16"
- board text added: "github.com/mar0x/patch_mate"
- board text removed: "2020.03.26"

Commit message: Updating voltage regulator part.
Parts:
- U2: value LM2575-5.0BU -> LM2576S-5.0
- U3: value LM2575-5.0BT -> LM2576HVT-5.0
Changed lines of the file:
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@@
       (effects (font (size 1 1) (thickness 0.15)))
     )
-    (fp_text value LM2575-5.0BU (at 0 6.65) (layer F.Fab)
+    (fp_text value LM2576S-5.0 (at 0 6.65) (layer F.Fab)
       (effects (font (size 1 1) (thickness 0.15)))
     )
@@
       (effects (font (size 1 1) (thickness 0.15)))
     )
-    (fp_text value LM2575-5.0BT (at 3.4 2.5 90) (layer F.Fab)
+    (fp_text value LM2576HVT-5.0 (at 3.4 2.5 90) (layer F.Fab)
       (effects (font (size 1 1) (thickness 0.15)))
     )
